Commit message: fix 2

File: ros2ws/src/ros2_gopigo3_node/urdf/gpg3_gopi5go_dave.urdf (robot description, URDF)
Before this commit: robot gopi5go_dave_v24_11_10, 10 links, 9 joints
Joints:
- joint joint_dave: origin xyz=-0.04 0 0.250 rpy=0 0 0 -> xyz=-0.04 0 0.2045615 rpy=0 0 0
- joint joint_dave_eyes: origin xyz=-0.04 0 0.250 rpy=0 0 0 -> xyz=-0.04 0 0.2045615 rpy=0 0 0

Commit message: appears to be right this time

File: ros2ws/src/ros2_gopigo3_node/urdf/gpg3_gopi5go_dave.urdf (robot description, URDF)
Before this commit: robot gopi5go_dave_v24_11_10, 10 links, 9 joints
Links:
- link base_link: mass 1.13 -> None

Commit message: move dave up

File: ros2ws/src/ros2_gopigo3_node/urdf/gpg3_gopi5go_dave.urdf (robot description, URDF)
Before this commit: robot gopi5go_dave_v24_11_10, 10 links, 9 joints
Joints:
- joint joint_dave: origin xyz=-0.04 0 0.2045615 rpy=0 0 0 -> xyz=-0.04 0 0.25 rpy=0 0 0

Commit message: imu lidar adj

File: ros2ws/src/ros2_gopigo3_node/urdf/gpg3_gopi5go_dave.urdf (robot description, URDF)
Before this commit: robot gopi5go_dave_v24_11_10, 10 links, 9 joints
Joints:
- joint joint_imu: origin xyz=0.070 0.035 0.104 rpy=0 0 0 -> xyz=0.070 0.035 0.0535615 rpy=0 0 0
- joint joint_ydlidar: origin xyz=-0.014 0 0.200 rpy=0 0 0 -> xyz=-0.014 0 0.1545615 rpy=0 0 0

Commit message: dave and cam

File: ros2ws/src/ros2_gopigo3_node/urdf/gpg3_gopi5go_dave.urdf (robot description, URDF)
Before this commit: robot gopi5go_dave_v24_11_10, 10 links, 9 joints
Joints:
- joint camera_joint: origin xyz=0.08 0 0.162 rpy=0 0 0 -> xyz=0.08 0 0.1165615 rpy=0 0 0
- joint joint_dave: origin xyz=-0.04 0 0.25 rpy=0 0 0 -> xyz=-0.04 0 0.2045615 rpy=0 0 0
